Commit message: refine k1 mesh

File: resources/robots/booster_robotics/K1/K1_22dof.urdf (robot description, URDF)
Before this commit: robot K1, 23 links, 22 joints
Links:
- link Head_1: geometry collision cylinder length=0.05 radius=0.03; visual mesh filename=meshes/Head_1.STL
- link Head_2: geometry collision box size=0.13 0.16 0.11; visual mesh filename=meshes/Head_2.STL
- link Left_Arm_3: geometry collision cylinder length=0.05 radius=0.03; collision cylinder length=0.09 radius=0.03
- link Right_Arm_3: geometry collision cylinder length=0.05 radius=0.03; collision cylinder length=0.09 radius=0.03
- link left_hand_link: geometry collision cylinder length=0.13 radius=0.02; collision sphere radius=0.027
- link right_hand_link: geometry collision cylinder length=0.13 radius=0.02; collision sphere radius=0.027

Commit message: refine k1 urdf

File: resources/robots/booster_robotics/K1/K1_22dof.urdf (robot description, URDF)
Before this commit: robot K1, 23 links, 22 joints
Links:
- link left_foot_link: geometry collision mesh filename=meshes/Left_Foot_Collision.STL; visual mesh filename=meshes/Left_Foot.STL
- link right_foot_link: geometry collision mesh filename=meshes/Right_Foot_Collision.STL; visual mesh filename=meshes/Right_Foot.STL
